Commit message: rm rviz

File: realsense2_camera/launch/d435_camera.urdf.xacro (robot description, xacro)
@@ -5,5 +5,5 @@
   <link name="base_link" />
   <xacro:sensor_d435 parent="base_link" use_nominal_extrinsics="$(arg use_nominal_extrinsics)">
-    <origin xyz="0 0 0" rpy="0 0 0"/>
+    <origin xyz="0 0 0.3" rpy="0 0 0"/>
   </xacro:sensor_d435>
 </robot>
